File: Battery-Controller.kicad_pcb (KiCad board)
At the start: 2 copper layers, 6 parts, among them U1 LM2674N-5.0, U2 DS1307+, U3 ADS1115IDGS

Commit message: Mise à jour empreintes
Parts:
- added BZ1: Buzzer, Buzzer_Beeper:Buzzer_12x9.5RM7.6, F.Cu at (162.3, 93.4)
- added C1: 100uF, Capacitor_Tantalum_SMD:CP_EIA-7260-20_AVX-M, F.Cu at (181.6, 100.4)
- added C2: 10nF, Capacitor_Tantalum_SMD:CP_EIA-7260-20_AVX-M, F.Cu at (191.2, 91.3)
- added C3: 0.1uF, Capacitor_Tantalum_SMD:CP_EIA-7260-20_AVX-M, F.Cu at (206.6, 81.1)
- added C4: 100uF, Capacitor_Tantalum_SMD:CP_EIA-7260-20_AVX-M, F.Cu at (207.3, 72.6)
- added D2: 4.7V, Diode_THT:D_A-405_P7.62mm_Horizontal, F.Cu at (187.9, 85.2)
- added D3: 4.7V, Diode_THT:D_A-405_P7.62mm_Horizontal, F.Cu at (204.0, 66.5)
- added D4: 4.7V, Diode_THT:D_A-405_P7.62mm_Horizontal, F.Cu at (152.7, 108.3)
- added D5: 4.7V, Diode_THT:D_A-405_P7.62mm_Horizontal, F.Cu at (200.7, 62.3)
- added D6: 1N5822, Diode_THT:D_5KP_P7.62mm_Vertical_AnodeUp, F.Cu at (189.2, 59.7)
- added D7: 1N5822, Diode_THT:D_DO-15_P10.16mm_Horizontal, F.Cu at (138.9, 107.1)
- added D8: 1N5822, Diode_THT:D_DO-15_P10.16mm_Horizontal, F.Cu at (163.2, 78.9)
- added D9: 1N5822, Diode_THT:D_DO-15_P10.16mm_Horizontal, F.Cu at (163.2, 84.1)
- added F1: Fuse, Fuse:Fuseholder_Blade_ATO_Littelfuse_Pudenz_2_Pin, F.Cu at (164.7, 51.6)
- added J1: Screw_Terminal_01x04 - RELAY, TerminalBlock_Phoenix:TerminalBlock_Phoenix_MKDS-1,5-4-5.08_1x04_P5.08mm_Horizontal, F.Cu at (131.5, 67.1)
- added J2: Screw_Terminal_01x04 - COM, TerminalBlock_Phoenix:TerminalBlock_Phoenix_MKDS-1,5-4-5.08_1x04_P5.08mm_Horizontal, F.Cu at (107.2, 90.2)
- added J3: Screw_Terminal_01x06 - RELAY STATUS, TerminalBlock_Phoenix:TerminalBlock_Phoenix_MKDS-1,5-6-5.08_1x06_P5.08mm_Horizontal, F.Cu at (107.2, 55.3)
- added J4: Screw_Terminal_01x02 - Battery IN, TerminalBlock_Phoenix:TerminalBlock_Phoenix_MKDS-1,5-2-5.08_1x02_P5.08mm_Horizontal, F.Cu at (181.5, 73.1)
- added J5: Screw_Terminal_01x02 - SOC Enable, TerminalBlock_Phoenix:TerminalBlock_Phoenix_MKDS-1,5-2-5.08_1x02_P5.08mm_Horizontal, F.Cu at (193.7, 71.5)
- added J6: Screw_Terminal_01x04 - Cells, TerminalBlock_Phoenix:TerminalBlock_Phoenix_MKDS-1,5-4-5.08_1x04_P5.08mm_Horizontal, F.Cu at (139.7, 55.3)
- added L1: 100uH, Inductor_THT:Choke_Schaffner_RN116-04-22.5x21.5mm, F.Cu at (105.9, 66.2)
- added Q1: TIP120, Package_TO_SOT_THT:TO-220-3_Vertical, F.Cu at (168.4, 104.1)
- added Q2: IRFZ44N, Package_TO_SOT_THT:TO-220-3_Vertical, F.Cu at (193.4, 81.1)
- added Q3: IRFZ44N, Package_TO_SOT_THT:TO-220-3_Vertical, F.Cu at (202.2, 58.1)
- added Q4: IRFZ44N, Package_TO_SOT_THT:TO-220-3_Vertical, F.Cu at (156.8, 104.1)
- added Q5: IRFZ44N, Package_TO_SOT_THT:TO-220-3_Vertical, F.Cu at (176.1, 94.4)
- added R1: 10K, Resistor_THT:R_Axial_DIN0411_L9.9mm_D3.6mm_P12.70mm_Horizontal, F.Cu at (128.0, 91.7)
- added R10: 1K, Resistor_THT:R_Axial_DIN0411_L9.9mm_D3.6mm_P12.70mm_Horizontal, F.Cu at (105.6, 108.7)
- added R11: 10K, Resistor_THT:R_Axial_DIN0411_L9.9mm_D3.6mm_P12.70mm_Horizontal, F.Cu at (122.3, 108.7)
- added R12: 10K, Resistor_THT:R_Axial_DIN0411_L9.9mm_D3.6mm_P12.70mm_Horizontal, F.Cu at (146.6, 80.5)
- added R13: 4.7K, Resistor_THT:R_Axial_DIN0411_L9.9mm_D3.6mm_P12.70mm_Horizontal, F.Cu at (144.6, 85.6)
- added R14: 10K, Resistor_THT:R_Axial_DIN0411_L9.9mm_D3.6mm_P12.70mm_Horizontal, F.Cu at (146.6, 75.3)
- added R15: 4.7K, Resistor_THT:R_Axial_DIN0411_L9.9mm_D3.6mm_P12.70mm_Horizontal, F.Cu at (152.3, 68.6)
- added R16: 10K, Resistor_THT:R_Axial_DIN0411_L9.9mm_D3.6mm_P12.70mm_Horizontal, F.Cu at (128.0, 86.5)
- added R17: 10K, Resistor_THT:R_Axial_DIN0411_L9.9mm_D3.6mm_P12.70mm_Horizontal, F.Cu at (105.6, 98.4)
- added R18: 10K, Resistor_THT:R_Axial_DIN0411_L9.9mm_D3.6mm_P12.70mm_Horizontal, F.Cu at (129.9, 75.3)
- added R19: 10K, Resistor_THT:R_Axial_DIN0411_L9.9mm_D3.6mm_P12.70mm_Horizontal, F.Cu at (105.6, 103.6)
- added R2: 4.7K, Resistor_THT:R_Axial_DIN0411_L9.9mm_D3.6mm_P12.70mm_Horizontal, F.Cu at (144.6, 90.8)
- added R20: 47, Resistor_THT:R_Axial_DIN0411_L9.9mm_D3.6mm_P12.70mm_Horizontal, F.Cu at (129.9, 80.5)
- added R21: 47, Resistor_THT:R_Axial_DIN0411_L9.9mm_D3.6mm_P12.70mm_Horizontal, F.Cu at (152.3, 63.5)
- added R22: 47, Resistor_THT:R_Axial_DIN0411_L9.9mm_D3.6mm_P12.70mm_Horizontal, F.Cu at (169.0, 59.2)
- added R23: 47, Resistor_THT:R_Axial_DIN0411_L9.9mm_D3.6mm_P12.70mm_Horizontal, F.Cu at (122.3, 103.6)
- added R3: 2.2K, Resistor_THT:R_Axial_DIN0411_L9.9mm_D3.6mm_P12.70mm_Horizontal, F.Cu at (163.2, 73.8)
- added R4: 10K, Resistor_THT:R_Axial_DIN0411_L9.9mm_D3.6mm_P12.70mm_Horizontal, F.Cu at (169.0, 64.3)
- added R5: 2.2K, Resistor_THT:R_Axial_DIN0411_L9.9mm_D3.6mm_P12.70mm_Horizontal, F.Cu at (138.9, 96.8)
- added R6: 2K, Resistor_THT:R_Axial_DIN0411_L9.9mm_D3.6mm_P12.70mm_Horizontal, F.Cu at (198.7, 51.6)
- added R7: 5.6K, Resistor_THT:R_Axial_DIN0411_L9.9mm_D3.6mm_P12.70mm_Horizontal, F.Cu at (138.9, 102.0)
- added R8: 1K, Resistor_THT:R_Axial_DIN0411_L9.9mm_D3.6mm_P12.70mm_Horizontal, F.Cu at (122.3, 98.4)
- added R9: 100, Resistor_THT:R_Axial_DIN0411_L9.9mm_D3.6mm_P12.70mm_Horizontal, F.Cu at (182.1, 51.6)
- added SW1: SW_DPST_x2, Connector_PinHeader_2.54mm:PinHeader_1x02_P2.54mm_Vertical, F.Cu at (199.5, 87.4)
- added U4: SN75176AP, Package_DIP:DIP-8_W7.62mm, F.Cu at (177.0, 80.8)
Connections:
- net GND renamed BAT-GND
- A2 pad 11: Net-(A2-Pad11) -> VICTRON-IN-1
- A2 pad 12: Net-(A2-Pad12) -> VICTRON-IN-2
- A2 pad 19: Net-(A2-Pad19) -> A0
- A2 pad 20: Net-(A2-Pad20) -> A1
- A2 pad 21: Net-(A2-Pad21) -> A2
- A2 pad 22: Net-(A2-Pad22) -> A3
- A2 pad 26: Net-(A2-Pad26) -> A7
- A2 pad 5: Net-(A2-Pad5) -> D2
- A2 pad 6: Net-(A2-Pad6) -> D3
- A2 pad 7: Net-(A2-Pad7) -> D4
- A2 pad 8: Net-(A2-Pad8) -> D5
- A2 pad 9: Net-(A2-Pad9) -> D6
- U1 pad 4: 5V -> +5V
- U1 pad 7: 12V -> BAT-12V
Other:
- net class power added: clearance 0.4, trace_width 1, via_dia 0.8, via_drill 0.4

Commit message: Mise en place composants
Parts:
- added J7: Conn_01x15_Male, Connector_PinHeader_2.54mm:PinHeader_1x15_P2.54mm_Vertical, F.Cu at (119.4, 177.8)
- added J8: Conn_01x15_Female, Connector_PinSocket_2.54mm:PinSocket_1x15_P2.54mm_Vertical, F.Cu at (121.9, 111.8)
- C1, C2, C3, C4: footprint Capacitor_Tantalum_SMD:CP_EIA-7260-20_AVX-M -> Capacitor_THT:C_Disc_D8.0mm_W5.0mm_P7.50mm
- D6: footprint Diode_THT:D_5KP_P7.62mm_Vertical_AnodeUp -> Diode_THT:D_DO-201AD_P15.24mm_Horizontal
- D7, D8, D9: footprint Diode_THT:D_DO-15_P10.16mm_Horizontal -> Diode_THT:D_DO-201AD_P15.24mm_Horizontal
- R1, R10, R11, R12, R13, R14, R15, R16, R17, R18, R19, R2, R20, R21, R22, R23, R3, R4, R5, R6, R7, R8, R9: footprint Resistor_THT:R_Axial_DIN0411_L9.9mm_D3.6mm_P12.70mm_Horizontal -> Resistor_THT:R_Axial_DIN0207_L6.3mm_D2.5mm_P10.16mm_Horizontal
- U3: footprint Package_SO:TSSOP-10_3x3mm_P0.5mm -> Charleslabs_Parts:ADC1115_ADC_Module
- moved D5 163.4 mm to (73.7, 165.1), turned to 270 degrees
- moved R6 159.7 mm to (86.4, 165.1), turned to 270 degrees
- moved R9 155.2 mm to (76.2, 165.1), turned to 270 degrees
- moved D3 150.8 mm to (83.8, 157.5), turned to 90 degrees
- moved C3 135.6 mm to (106.7, 172.7)
- moved D2 135.2 mm to (73.7, 157.5), turned to 90 degrees
- moved R4 127.9 mm to (81.3, 157.5), turned to 90 degrees
- moved C4 124.4 mm to (86.4, 43.2)
- moved R3 122.7 mm to (81.3, 165.1), turned to 270 degrees
- moved A1 107.4 mm to (144.8, 154.9)
- moved C1 107.4 mm to (86.4, 50.8)
- moved C2 101.8 mm to (94.0, 61.0)
- moved SW1 101.1 mm to (99.1, 99.1), turned to 180 degrees
- moved J6 95.1 mm to (91.4, 137.2), turned to 180 degrees
- moved R5 91.0 mm to (71.1, 157.5), turned to 90 degrees
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Connections:
- A1 pad 1: +3V3 -> TUP-02
- A1 pad 2: D10 -> UP-CS
- A1 pad 3: D11 -> UP-MOSI
- A1 pad 4: D13 -> UP-CLK
- A1 pad 5: D12 -> UP-MISO
- A1 pad 6: BAT-GND -> TUP-01
- A2 pad 11: VICTRON-IN-1 -> D8
- A2 pad 12: VICTRON-IN-2 -> D9
- C3 pad 2: BAT-GND -> TUP-01
- D2 pad 2: BAT-GND -> TUP-01
- D3 pad 2: BAT-GND -> TUP-01
- D4 pad 2: BAT-GND -> TUP-01
- D5 pad 2: BAT-GND -> TUP-01
- R11 pad 1: BAT-GND -> TUP-01
- R6 pad 2: BAT-GND -> TUP-01
- R7 pad 2: BAT-GND -> TUP-01
- R8 pad 2: BAT-GND -> TUP-01
- U2 pad 4: BAT-GND -> TUP-01
- U2 pad 5: SDA -> UP-SDA
- U2 pad 6: SCL -> UP-SCL
- U2 pad 8: +5V -> TUP-02
- U3 pad 10: SCL -> UP-SCL
- U3 pad 3: BAT-GND -> TUP-01
- U3 pad 9: SDA -> UP-SDA
- U4 pad 1: D3 -> UP-D3
- U4 pad 4: D2 -> UP-D2
