File: Battery-Controller.sch (KiCad schematic (older format))
At the start: 57 parts, among them Q1 Q_NPN_BCE, SW1 SW_DPST_x2, U1 LM2674N-5.0, U2 DS1307+, U3 ADS1115IDGS

Commit message: Mise à jour empreintes
Parts:
- D2, D3, D4, D5: renamed from D?; footprint (none) -> Diode_THT:D_A-405_P7.62mm_Horizontal
- D6: renamed from D?; footprint Diode_THT:D_DO-201AD_P15.24mm_Horizontal -> Diode_THT:D_5KP_P7.62mm_Vertical_AnodeUp
- D7, D8, D9: renamed from D?; footprint Diode_THT:D_DO-201AD_P15.24mm_Horizontal -> Diode_THT:D_DO-15_P10.16mm_Horizontal
- J1, J2, J6: renamed from J?; footprint (none) -> TerminalBlock_Phoenix:TerminalBlock_Phoenix_MKDS-1,5-4-5.08_1x04_P5.08mm_Horizontal
- J3: renamed from J?; footprint (none) -> TerminalBlock_Phoenix:TerminalBlock_Phoenix_MKDS-1,5-6-5.08_1x06_P5.08mm_Horizontal
- J4, J5: renamed from J?; footprint (none) -> TerminalBlock_Phoenix:TerminalBlock_Phoenix_MKDS-1,5-2-5.08_1x02_P5.08mm_Horizontal
- Q1: value Q_NPN_BCE -> TIP120; footprint (none) -> Package_TO_SOT_THT:TO-220-3_Vertical; symbol Device:Q_NPN_BCE -> Transistor_BJT:TIP120
- Q2, Q3, Q4, Q5: renamed from Q?; footprint Package_DirectFET:DirectFET_ST -> Package_TO_SOT_THT:TO-220-3_Vertical
- R1, R10: footprint (none) -> Resistor_THT:R_Axial_DIN0411_L9.9mm_D3.6mm_P12.70mm_Horizontal
- R11, R12, R13, R14, R15, R16, R17, R18, R19, R2, R20, R21, R22, R23, R3, R4, R5, R6, R7, R8, R9: renamed from R?; footprint (none) -> Resistor_THT:R_Axial_DIN0411_L9.9mm_D3.6mm_P12.70mm_Horizontal
- SW1: footprint (none) -> Connector_PinHeader_2.54mm:PinHeader_1x02_P2.54mm_Vertical
- gave numbers to parts that had none: 1

Commit message: Mise en place composants
Parts:
- added J7: Conn_01x15_Male, Connector_PinHeader_2.54mm:PinHeader_1x15_P2.54mm_Vertical, symbol Connector:Conn_01x15_Male
- added J8: Conn_01x15_Female, Connector_PinSocket_2.54mm:PinSocket_1x15_P2.54mm_Vertical, symbol Connector:Conn_01x15_Female
- C1, C2, C3, C4: footprint Capacitor_Tantalum_SMD:CP_EIA-7260-20_AVX-M -> Capacitor_THT:C_Disc_D8.0mm_W5.0mm_P7.50mm
- D6: footprint Diode_THT:D_5KP_P7.62mm_Vertical_AnodeUp -> Diode_THT:D_DO-201AD_P15.24mm_Horizontal
- D7, D8, D9: footprint Diode_THT:D_DO-15_P10.16mm_Horizontal -> Diode_THT:D_DO-201AD_P15.24mm_Horizontal
- R1, R10, R11, R12, R13, R14, R15, R16, R17, R18, R19, R2, R20, R21, R22, R23, R3, R4, R5, R6, R7, R8, R9: footprint Resistor_THT:R_Axial_DIN0411_L9.9mm_D3.6mm_P12.70mm_Horizontal -> Resistor_THT:R_Axial_DIN0207_L6.3mm_D2.5mm_P10.16mm_Horizontal
- U3: footprint Package_SO:TSSOP-10_3x3mm_P0.5mm -> Charleslabs_Parts:ADC1115_ADC_Module
Connections:
- net labels added: +3.3VA, +5VD, D8, D9, GND2, TUP-01, TUP-02, UP-CLK, UP-CS, UP-D2, UP-D3, UP-MISO, UP-MOSI, UP-SCL, UP-SDA
- net labels removed: +3.3V
- wire segments 112 -> 124
Other:
- note added: "Connecteur Femelle \nPCB Inférieur\n"
- note added: "Connecteur Male \nPCB supérieur"
- moved on the sheet: A1
