File: kicad/Battery-Controller.sch (KiCad schematic (older format))
At the start: 59 parts, among them J1 Screw_Terminal_01x04 - RELAY, J2 Screw_Terminal_01x04 - COM, J3 Screw_Terminal_01x06 - RELAY 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, J4 Screw_Terminal_01x02 - Batter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, J5 Screw_Terminal_01x02 - SOC En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, J6 Screw_Terminal_01x04 - Cells, J7 Conn_01x15_Male, J8 Conn_01x15_Female, Q1 TIP120, Q2 IRFZ44N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

Commit message: Ajout logs SD Card
Parts:
- removed C1, C4: 100uF, Capacitor_THT:C_Disc_D8.0mm_W5.0mm_P7.50mm, symbol Device:CP
- removed C2: 10nF, Capacitor_THT:C_Disc_D8.0mm_W5.0mm_P7.50mm, symbol Device:C
- removed D2, D3, D4, D5: 4.7V, Diode_THT:D_A-405_P7.62mm_Horizontal, symbol Diode:DZ2S047X0L
- removed L1: 100uH, Inductor_THT:Choke_Schaffner_RN116-04-22.5x21.5mm, symbol pspice:INDUCTOR
- removed R9: 100, Resistor_THT:R_Axial_DIN0207_L6.3mm_D2.5mm_P10.16mm_Horizontal, symbol Device:R
- removed U1: LM2674N-5.0, Package_DIP:DIP-8_W7.62mm, symbol Regulator_Switching:LM2674N-5.0
- added U1: YAAJ_DCDC_StepDown_LM2596, DC_DC_LM2596:YAAJ_DCDC_StepDown_LM2596, symbol yaaj_dcdc_stepdown_lm2596:YAAJ_DCDC_StepDown_LM2596
- D6: footprint Diode_THT:D_5KP_P7.62mm_Vertical_AnodeUp -> Diode_THT:D_5W_P5.08mm_Vertical_AnodeUp
- D7, D8, D9: footprint Diode_THT:D_DO-15_P10.16mm_Horizontal -> Diode_THT:D_5W_P5.08mm_Vertical_AnodeUp
- R3: value 2.2K -> 21.6K
- R4: value 10K -> 474
- R5: value 2.2K -> 5.1K
- R6: value 2K -> 32K
- R7: value 5.6K -> 330
- R8: value 1K -> 2.2K
Connections:
- net labels added: UP-3.3V, UP-5V, UP-D7
- wire segments 124 -> 95
Other:
- note added: "10.95V"
- note added: "14.6V"
- note added: "3.65V"
- note added: "7.3V"
- note added: "DC-DC Converter\nFrom 12V to 5V"
- note added: "Low side relay"
- note removed: "Alimentation 5V\nOutput 5V 500mA\nInput 7-40V"
- moved on the sheet: D6, D7, D8

Commit message: Calibration entrées Cells
Parts:
- removed J5: Screw_Terminal_01x02 - SOC Enable, TerminalBlock_Phoenix:TerminalBlock_Phoenix_MKDS-1,5-2-5.08_1x02_P5.08mm_Horizontal, symbol Connector:Screw_Terminal_01x02
- J3: value Screw_Terminal_01x06 - RELAY STATUS -> Screw_Terminal_01x08 - RELAY STATUS; footprint TerminalBlock_Phoenix:TerminalBlock_Phoenix_MKDS-1,5-6-5.08_1x06_P5.08mm_Horizontal -> TerminalBlock_Phoenix:TerminalBlock_Phoenix_MKDS-1,5-7-5.08_1x07_P5.08mm_Horizontal; symbol Connector:Screw_Terminal_01x06 -> Connector:Screw_Terminal_01x08
Connections:
- wire segments 95 -> 94
Other:
- moved on the sheet: J4
Changed lines of the file:
@@
 	1    0    0    -1
 $EndComp
-Text GLabel 9900 2300 0    50   Input ~ 0
+Text GLabel 9900 2350 0    50   Input ~ 0
 CHARGING-STATUS
 $Comp
@@
 	750  7050 2500 7050
 $Comp
-L Connector:Screw_Terminal_01x06 J3
+L Connector:Screw_Terminal_01x08 J3
 U 1 1 61D0860E
-P 10100 2100
-F 0 "J3" H 10180 2092 50  0000 L CNN
-F 1 "Screw_Terminal_01x06 - RELAY STATUS" H 10180 2001 50  0000 L CNN
-F 2 "TerminalBlock_Phoenix:TerminalBlock_Phoenix_MKDS-1,5-6-5.08_1x06_P5.08mm_Horizontal" H 10100 2100 50  0001 C CNN
-F 3 "~" H 10100 2100 50  0001 C CNN
-	1    10100 2100
-	1    0    0    -1
-$EndComp
-Text GLabel 9900 2200 0    50   Input ~ 0
+P 10100 2250
+F 0 "J3" H 10180 2242 50  0000 L CNN
+F 1 "Screw_Terminal_01x08 - RELAY STATUS" H 10180 2151 50  0000 L CNN
+F 2 "TerminalBlock_Phoenix:TerminalBlock_Phoenix_MKDS-1,5-7-5.08_1x07_P5.08mm_Horizontal" H 10100 2250 50  0001 C CNN
+F 3 "~" H 10100 2250 50  0001 C CNN
+	1    10100 2250
+	1    0    0    -1
+$EndComp
+Text GLabel 9900 2150 0    50   Input ~ 0
 THERMOCOUPLE-IN-N
 Text GLabel 1750 7700 0    50   Input ~ 0
@@
 L Connector:Screw_Terminal_01x02 J4
 U 1 1 61D1C628
-P 10100 2600
-F 0 "J4" H 10180 2592 50  0000 L CNN
-F 1 "Screw_Terminal_01x02 - Battery IN" H 10180 2501 50  0000 L CNN
-F 2 "TerminalBlock_Phoenix:TerminalBlock_Phoenix_MKDS-1,5-2-5.08_1x02_P5.08mm_Horizontal" H 10100 2600 50  0001 C CNN
-F 3 "~" H 10100 2600 50  0001 C CNN
-	1    10100 2600
-	1    0    0    -1
-$EndComp
-Text GLabel 9900 2600 0    50   Input ~ 0
-BAT-12V
-Text GLabel 9900 2700 0    50   Input ~ 0
+P 10100 2900
+F 0 "J4" H 10180 2892 50  0000 L CNN
+F 1 "Screw_Terminal_01x02 - Battery IN" H 10180 2801 50  0000 L CNN
+F 2 "TerminalBlock_Phoenix:TerminalBlock_Phoenix_MKDS-1,5-2-5.08_1x02_P5.08mm_Horizontal" H 10100 2900 50  0001 C CNN
+F 3 "~" H 10100 2900 50  0001 C CNN
+	1    10100 2900
+	1    0    0    -1
+$EndComp
+Text GLabel 9900 2900 0    50   Input ~ 0
+BAT-12V
+Text GLabel 9900 3000 0    50   Input ~ 0
 BAT-GND
 Text GLabel 1400 2600 0    50   Input ~ 0
@@
 Text GLabel 13450 2350 0    50   Input ~ 0
 VICTRON-IN-2
-Text GLabel 9900 2100 0    50   Input ~ 0
+Text GLabel 9900 2250 0    50   Input ~ 0
 THERMOCOUPLE-IN-P
 Text GLabel 6500 1000 0    50   Input ~ 0
@@
 Wire Notes Line
 	5450 700  8150 700
-Text GLabel 9900 1900 0    50   Input ~ 0
+Text GLabel 9900 1950 0    50   Input ~ 0
 CHARGE-RELAY-STATUS
-Text GLabel 9900 2000 0    50   Input ~ 0
+Text GLabel 9900 2050 0    50   Input ~ 0
 LOAD-RELAY-STATUS
 Wire Wire Line
@@
 Wire Wire Line
 	6800 7800 6750 7800
-Text GLabel 9900 2900 0    50   Input ~ 0
+Text GLabel 9900 2550 0    50   Input ~ 0
 SOC-ENABLE
 Text GLabel 1350 8400 0    50   Input ~ 0
@@
 SOC ON/OFF Bouton
 $Comp
-L Connector:Screw_Terminal_01x02 J5
-U 1 1 61D8E185
-P 10100 2900
-F 0 "J5" H 10180 2892 50  0000 L CNN
-F 1 "Screw_Terminal_01x02 - SOC Enable" H 10180 2801 50  0000 L CNN
-F 2 "TerminalBlock_Phoenix:TerminalBlock_Phoenix_MKDS-1,5-2-5.08_1x02_P5.08mm_Horizontal" H 10100 2900 50  0001 C CNN
-F 3 "~" H 10100 2900 50  0001 C CNN
-	1    10100 2900
-	1    0    0    -1
-$EndComp
-$Comp
-L power:+5V #PWR0137
-U 1 1 61D8F291
-P 9250 3000
-F 0 "#PWR0137" H 9250 2850 50  0001 C CNN
-F 1 "+5V" H 9265 3173 50  0000 C CNN
-F 2 "" H 9250 3000 50  0001 C CNN
-F 3 "" H 9250 3000 50  0001 C CNN
-	1    9250 3000
-	1    0    0    -1
-$EndComp
-Wire Wire Line
-	9250 3000 9900 3000
-$Comp
 L Connector:Screw_Terminal_01x04 J6
 U 1 1 61DEB6EA
@@
 	1    0    0    -1
 $EndComp
-Text GLabel 9900 3200 0    50   Input ~ 0
-CELL-1
 Text GLabel 9900 3300 0    50   Input ~ 0
 CELL-2
@@
 Text Notes 1800 4600 0    50   ~ 0
 14.6V
+Text GLabel 9900 3200 0    50   Input ~ 0
+CELL-1
+Text GLabel 9900 2450 0    50   Input ~ 0
+5V
 $EndSCHEMATC

Commit message: Intégration des routines de surveillance de la température
Parts:
- J3: value Screw_Terminal_01x08 - RELAY STATUS -> Screw_Terminal_01x08; footprint TerminalBlock_Phoenix:TerminalBlock_Phoenix_MKDS-1,5-7-5.08_1x07_P5.08mm_Horizontal -> TerminalBlock_Phoenix:TerminalBlock_Phoenix_MKDS-1,5-8-5.08_1x08_P5.08mm_Horizontal
Connections:
- net labels added: HREF
- net labels removed: +5V
- wire segments 94 -> 98
Changed lines of the file:
@@
 	0    -1   -1   0
-$EndComp
-$Comp
-L power:+5V #PWR0125
-U 1 1 61BBF6FB
-P 2250 7400
-F 0 "#PWR0125" H 2250 7250 50  0001 C CNN
-F 1 "+5V" H 2265 7573 50  0000 C CNN
-F 2 "" H 2250 7400 50  0001 C CNN
-F 3 "" H 2250 7400 50  0001 C CNN
-	1    2250 7400
-	1    0    0    -1
 $EndComp
 Wire Wire Line
@@
 Text GLabel 1750 7400 0    50   Input ~ 0
 THERMOCOUPLE-IN-P
-Wire Notes Line
-	750  7050 2500 7050
 $Comp
 L Connector:Screw_Terminal_01x08 J3
@@
 P 10100 2250
 F 0 "J3" H 10180 2242 50  0000 L CNN
-F 1 "Screw_Terminal_01x08 - RELAY STATUS" H 10180 2151 50  0000 L CNN
-F 2 "TerminalBlock_Phoenix:TerminalBlock_Phoenix_MKDS-1,5-7-5.08_1x07_P5.08mm_Horizontal" H 10100 2250 50  0001 C CNN
+F 1 "Screw_Terminal_01x08" H 10180 2151 50  0000 L CNN
+F 2 "TerminalBlock_Phoenix:TerminalBlock_Phoenix_MKDS-1,5-8-5.08_1x08_P5.08mm_Horizontal" H 10100 2250 50  0001 C CNN
 F 3 "~" H 10100 2250 50  0001 C CNN
 	1    10100 2250
@@
 Wire Wire Line
 	1900 7700 1750 7700
-Wire Notes Line
-	2500 8100 750  8100
-Wire Notes Line
-	2500 7050 2500 8100
 Wire Notes Line
 	750  7050 750  8100
@@
 Text GLabel 9900 2450 0    50   Input ~ 0
 5V
+Text GLabel 2350 7400 2    50   Input ~ 0
+3.3V
+Text GLabel 2350 7550 2    50   Input ~ 0
+HREF
+Wire Wire Line
+	2200 7400 2250 7400
+Wire Wire Line
+	2250 7400 2350 7400
+Connection ~ 2250 7400
+Wire Wire Line
+	2350 7550 2250 7550
+Wire Wire Line
+	2250 7550 2250 7400
+Wire Notes Line
+	2700 7050 2700 8100
+Wire Notes Line
+	750  7050 2700 7050
+Wire Notes Line
+	750  8100 2700 8100
 $EndSCHEMATC

Commit message: Optimisation du code
Parts:
- removed D7, D8, D9: 1N5822, Diode_THT:D_5W_P5.08mm_Vertical_AnodeUp, symbol Diode:1N5822
- removed Q2, Q3, Q4, Q5: IRFZ44N, Package_TO_SOT_THT:TO-220-3_Vertical, symbol IRFZ44N:IRFZ44N
- added D2, D3, D4: 1N5822, Diode_THT:D_5W_P5.08mm_Vertical_AnodeUp, symbol Diode:1N5822
- added Q2, Q3, Q4, Q5: TIP122, Package_TO_SOT_THT:TO-220-3_Vertical, symbol Transistor_BJT:TIP122
- added Q6, Q7, Q8, Q9: TIP42C, Package_TO_SOT_THT:TO-220-3_Vertical, symbol Transistor_BJT:TIP42C
- added R24: 1K, Resistor_THT:R_Axial_DIN0207_L6.3mm_D2.5mm_P10.16mm_Horizontal, symbol Device:R
- added R9: 10K, Resistor_THT:R_Axial_DIN0207_L6.3mm_D2.5mm_P10.16mm_Horizontal, symbol Device:R
- R12: value 10K -> 1K; Field4 (none) -> Limit gate current
- R13, R15: value 4.7K -> 1K; Field4 (none) -> Limit gate current
- R16, R18: value 10K -> 1K
- R17, R19: value 10K -> 1K; Field4 (none) -> Pull down in case pin hi-impedence
- R20, R22: value 47 -> 1K
- R21, R23: value 47 -> 1K; Field4 (none) -> Limit gate current
Connections:
- wire segments 98 -> 112
Other:
- note added: "HIGH side relay"
- moved on the sheet: D6, R16, R20
